File: singleDriverJaredSchein.kicad_pcb (KiCad board)
At the start: 2 copper layers, 30 parts, among them J1 Conn_01x02_Pin, J2 Conn_01x04_Pin, J3 conn01x12, J4 Conn_01x02_Pin, U1 DRV10970

Commit message: Add files via upload
Parts:
- removed TP1: FG, TestPoint:TestPoint_Keystone_5019_Minature
- removed TP10: U_HP, TestPoint:TestPoint_Keystone_5019_Minature
- removed TP11: V_HN, TestPoint:TestPoint_Keystone_5019_Minature
- removed TP12: W_HN, TestPoint:TestPoint_Keystone_5019_Minature
- removed TP13: V_HP, TestPoint:TestPoint_Keystone_5019_Minature
- removed TP2: RD, TestPoint:TestPoint_Keystone_5019_Minature
- removed TP33: DAA, TestPoint:TestPoint_Keystone_5019_Minature
- removed TP9: W_HP, TestPoint:TestPoint_Keystone_5019_Minature
Routing:
- net Net-(J3-Hall_Sensor_Abar): track 41.6 -> 79.7 mm, vias 5 -> 4
- net Net-(J3-Hall_Sensor_Bbar): track 39.4 -> 68.9 mm, vias 1 -> 2
- net Net-(U1-DAA): track 27.2 -> 0.00 mm, vias 2 -> 0
- net /FG: track 25.0 -> 44.2 mm, vias 2 -> 4
- net Net-(J3-Hall_Sensor_B): track 33.1 -> 48.7 mm, vias 2 -> 5
- net /VINT: track 41.1 -> 54.5 mm
- net GND: track 8.06 -> 15.0 mm, vias 2 -> 5
- net Net-(J3-Hall_Sensor_A): track 55.3 -> 49.2 mm, vias 0 -> 4
- net Net-(J3-Hall_Sensor_Cbar): track 58.4 -> 55.6 mm
- net /PWM: track 29.7 -> 29.0 mm
- net Net-(J3-Hall_Sensor_C): track 83.9 -> 84.5 mm
- net Net-(U1-CS): track 9.72 -> 10.2 mm
Other:
- board outline added: 53.3 x 38.1 mm
